File: _autosave-PCB_Banc.kicad_sch (KiCad schematic)
At the start: 29 parts, among them J1 Screw_Terminal_01x08, J2 Screw_Terminal_01x08, J3 Screw_Terminal_01x02, J4 Screw_Terminal_01x02, J5 Screw_Terminal_01x02, J6 Screw_Terminal_01x02, J7 Screw_Terminal_01x02, Q1 IRLZ44N, Q2 IRLZ44N, Q3 IRLZ44N, Q4 IRLZ44N

Commit message: alim
Parts:
- added C3: 470µ, symbol Device:C
- added C4: 100n, symbol Device:C
Connections:
- net +24V: now also D1.1 (K), D4.1 (K), D6.1 (K), D8.1 (K), J1.8 (Pin_8), J3.1 (Pin_1), J4.1 (Pin_1), J5.1 (Pin_1), J6.1 (Pin_1), R2.1, R3.1, R5.1, R7.1, C3.1, C4.1
- net GND: now also C3.2, C4.2; no longer J1.2 (Pin_2), J1.4 (Pin_4), J1.6 (Pin_6), J1.8 (Pin_8)
- now unconnected: J1.1 (Pin_1), J1.3 (Pin_3), J1.5 (Pin_5), J1.7 (Pin_7)
Other:
- moved on the sheet: D1, D4, D6, D8, J2, J3, J4, J5, J6, Q1, Q2, Q3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

Commit message: before edit
Parts:
- removed C3: 470µ, symbol Device:C
- removed C4: 100n, symbol Device:C
- removed J1: Screw_Terminal_01x08, symbol Connector:Screw_Terminal_01x08
Other:
- moved on the sheet: C1, C2

Commit message: next step
Parts:
- added A1: Pololu_Breakout_A4988, Module:Pololu_Breakout-16_15.2x20.3mm, symbol Driver_Motor:Pololu_Breakout_A4988
- added J1: Screw_Terminal_01x02, symbol Connector:Screw_Terminal_01x02
- added R10, R11, R9: 10K, Resistor_THT:R_Axial_DIN0411_L9.9mm_D3.6mm_P12.70mm_Horizontal, symbol Device:R
- added U1: LM358, symbol Amplifier_Operational:LM358
- added U2: MAX232, symbol Interface_UART:MAX232
Connections:
- net GND: now also J1.1 (Pin_1), R10.2
- new net: J1.2 (Pin_2), R9.1
- new net: R9.2, U1.3 (+)
- new net: R10.1, R11.1, U1.2 (-)
- new net: R11.2, U1.1
Other:
- note added: "0-10V PWM (J1 from CPU Unit 5v)"
- note added: "4-20ma"
- note added: "RS232"
- note added: "RS485"
- note added: "pas à pas"
- moved on the sheet: C1, C2, J7

Commit message: before rs485
Parts:
- added C3: C, symbol Device:C
- added C4, C5, C6, C7, C8: 2.2µF, symbol Device:C_Polarized
- added J10, J12: Screw_Terminal_01x02, symbol Connector:Screw_Terminal_01x02
- added J11: DE9_Plug, symbol Connector:DE9_Plug
- added J14, J9: Screw_Terminal_01x04, symbol Connector:Screw_Terminal_01x04
- added J8: Screw_Terminal_01x06, symbol Connector:Screw_Terminal_01x06
- added R12, R13, R14, R15: 10K, Resistor_THT:R_Axial_DIN0411_L9.9mm_D3.6mm_P12.70mm_Horizontal, symbol Device:R
- added U3: LM358, symbol Amplifier_Operational:LM358
- added U4: MAX1487E, Package_SO:SOIC-8_3.9x4.9mm_P1.27mm, symbol Interface_UART:MAX1487E
Connections:
- net +24V: now also A1.2 (VDD)
- net GND: now also A1.7 (GND), U2.15 (GND), C3.2, C6.1, C8.2, J10.1 (Pin_1), J11.5, R13.2, U4.5 (GND)
- net at R9.1: now also C3.1, R15.2; no longer J1.2 (Pin_2)
- net at A1.1 (GND): now also J8.1 (Pin_1)
- net at A1.10 (MS1): now also J8.3 (Pin_3)
- net at A1.11 (MS2): now also J8.2 (Pin_2)
- net at A1.15 (STEP): now also J8.5 (Pin_5)
- net at A1.16 (DIR): now also J8.4 (Pin_4)
- net at A1.3 (1B): now also J9.1 (Pin_1)
- net at A1.4 (1A): now also J9.2 (Pin_2)
- net at A1.5 (2A): now also J9.3 (Pin_3)
- net at A1.6 (2B): now also J9.4 (Pin_4)
- net at A1.9 (~{ENABLE}): now also J8.6 (Pin_6)
- net at U2.1 (C1+): now also C4.1
- net at U2.11 (T1IN): now also J12.2 (Pin_2)
- net at U2.12 (R1OUT): now also J12.1 (Pin_1)
- net at U2.13 (R1IN): now also J11.3
- net at U2.14 (T1OUT): now also J11.2
- net +5V: now reaches U2.16 (VCC)
- net +5V: now also C7.2, C8.1
- net at U2.2 (VS+): now also C7.1
- net at U2.3 (C1-): now also C4.2
- net at U2.4 (C2+): now also C5.1
- net at U2.5 (C2-): now also C5.2
- net at U2.6 (VS-): now also C6.2
- new net: R13.1, R14.1, U3.2 (-)
- new net: R14.2, U3.1
- new net: J1.2 (Pin_2), R15.1
- new net: R12.2, U3.3 (+)
- new net: J10.2 (Pin_2), R12.1
- new net: J14.4 (Pin_4), U4.1 (RO)
- new net: J14.3 (Pin_3), U4.2 (~{RE})
- new net: J14.2 (Pin_2), U4.3 (DE)
- new net: J14.1 (Pin_1), U4.4 (DI)
Other:
- note added: "0-10V DC (J1 from CPU Unit PWM 10KHz)"
- note added: "0-10V PWM (J1 from CPU Unit)"
- note added: "Pilotage moteurs pas à pas"
- note added: "UART_RX"
- note added: "UART_TX"
- note removed: "0-10V PWM (J1 from CPU Unit 5v)"
- note removed: "pas à pas"
- moved on the sheet: A1, C1, C2, J1, J7, R10, R11, R9, U1A, U2
