File: PCB_Banc.kicad_sch (KiCad schematic)
At the start: 7 parts, among them J1 Conn_01x02_Pin, J2 Conn_01x02_Pin, Q1 IRLZ44N

Commit message: saving
Parts:
- removed D1: 1N4001, Diode_THT:D_DO-41_SOD81_P10.16mm_Horizontal, symbol Diode:1N4001
- removed D2: LED, symbol Device:LED
- removed J1, J2: Conn_01x02_Pin, Connector_PinHeader_2.54mm:PinHeader_2x01_P2.54mm_Vertical, symbol Connector:Conn_01x02_Pin
- added A1, A2, A3, A4: Pololu_Breakout_A4988, Module:Pololu_Breakout-16_15.2x20.3mm, symbol Driver_Motor:Pololu_Breakout_A4988
- added C1: 0.33µF, Capacitor_THT:CP_Axial_L10.0mm_D4.5mm_P15.00mm_Horizontal, symbol Device:C
- added C10, C7: ~, symbol Device:C
- added C11, C12, C13, C8, C9: 2.2µF, symbol Device:C_Polarized
- added C14: 2.2µF, symbol Device:C
- added C15: 100nF, symbol Device:C
- added C2: 470µ, symbol Device:C
- added C3, C6: 47µ, symbol Device:C
- added C4: 100n, symbol Device:C
- added C5: 0.1µ, symbol Device:C
- added D1, D10, D3, D5, D7, D9: LED, LED_SMD:LED_0201_0603Metric_Pad0.64x0.40mm_HandSolder, symbol Device:LED
- added D2, D4, D6: 1N4001, Diode_SMD:D_0805_2012Metric, symbol Diode:1N4001
- added D8: 1N4001, Diode_SMD:D_0805_2012Metric_Pad1.15x1.40mm_HandSolder, symbol Diode:1N4001
- added J1, J10, J12, J13, J15, J16, J2, J25, J26, J3, J4, J6, J7, J9: Screw_Terminal_01x02, TerminalBlock_Phoenix:TerminalBlock_Phoenix_MPT-0,5-2-2.54_1x02_P2.54mm_Horizontal, symbol Connector:Screw_Terminal_01x02
- added J11, J14, J20, J21, J22, J27, J28: Screw_Terminal_01x04, TerminalBlock_Phoenix:TerminalBlock_Phoenix_MPT-0,5-4-2.54_1x04_P2.54mm_Horizontal, symbol Connector:Screw_Terminal_01x04
- added J17, J18, J23, J24: Screw_Terminal_01x06, TerminalBlock_Phoenix:TerminalBlock_Phoenix_MPT-0,5-6-2.54_1x06_P2.54mm_Horizontal, symbol Connector:Screw_Terminal_01x06
- added J19: DE9_Plug, symbol Connector:DE9_Plug
- added J5: Arduino pwr supply, TerminalBlock_Phoenix:TerminalBlock_Phoenix_MPT-0,5-2-2.54_1x02_P2.54mm_Horizontal, symbol Connector:Screw_Terminal_01x02
- added J8: Screw_Terminal_01x08, TerminalBlock_Phoenix:TerminalBlock_Phoenix_MPT-0,5-8-2.54_1x08_P2.54mm_Horizontal, symbol Connector:Screw_Terminal_01x08
- added Q2, Q3, Q4: IRLZ44N, Package_TO_SOT_THT:TO-220-3_Vertical, symbol Transistor_FET:IRLZ44N
- added R10, R5: 10K, Resistor_SMD:R_0805_2012Metric, symbol Device:R
- added R11, R12: 1K, Resistor_THT:R_Axial_DIN0411_L9.9mm_D3.6mm_P12.70mm_Horizontal, symbol Device:R
- added R13, R14, R15, R16, R20, R21, R23: 5k, Resistor_THT:R_Axial_DIN0411_L9.9mm_D3.6mm_P12.70mm_Horizontal, symbol Device:R
- added R17: 200, Resistor_THT:R_Axial_DIN0411_L9.9mm_D3.6mm_P12.70mm_Horizontal, symbol Device:R
- added R18, R19, R22: 5k, Resistor_SMD:R_0805_2012Metric_Pad1.20x1.40mm_HandSolder, symbol Device:R
- added R24: 470, Resistor_SMD:R_0805_2012Metric_Pad1.20x1.40mm_HandSolder, symbol Device:R
- added R25: 2k, Resistor_SMD:R_0805_2012Metric_Pad1.20x1.40mm_HandSolder, symbol Device:R
- added R3, R7: 247, Resistor_THT:R_Axial_DIN0411_L9.9mm_D3.6mm_P12.70mm_Horizontal, symbol Device:R
- added R4: 130, Resistor_SMD:R_0805_2012Metric_Pad1.20x1.40mm_HandSolder, symbol Device:R
- added R6, R9: 130, Resistor_SMD:R_0805_2012Metric, symbol Device:R
- added R8: 10K, Resistor_SMD:R_0805_2012Metric_Pad1.20x1.40mm_HandSolder, symbol Device:R
- added U1: L7805, Package_TO_SOT_THT:TO-220-3_Vertical, symbol Regulator_Linear:L7805
- added U2: XTR111AxDGQ, Package_SO:MSOP-10-1EP_3x3mm_P0.5mm_EP2.2x3.1mm_Mask1.83x1.89mm_ThermalVias, symbol Interface_CurrentLoop:XTR111AxDGQ
- added U3: MAX232, symbol Interface_UART:MAX232
- added U4: MAX1487E, Package_SO:SOIC-8_3.9x4.9mm_P1.27mm, symbol Interface_UART:MAX1487E
- added U5, U6: LM358, symbol Amplifier_Operational:LM358
- R1: value 10K -> 130; footprint Resistor_THT:R_Axial_DIN0411_L9.9mm_D3.6mm_P12.70mm_Horizontal -> Resistor_SMD:R_0805_2012Metric_Pad1.20x1.40mm_HandSolder
- R2: value 130 -> 10K; footprint Resistor_THT:R_Axial_DIN0411_L9.9mm_D3.6mm_P12.70mm_Horizontal -> Resistor_SMD:R_0805_2012Metric_Pad1.20x1.40mm_HandSolder
Connections:
- net +24V: now also R1.1, C1.1, C2.1, C4.1, D2.1 (K), D4.1 (K), D6.1 (K), D8.1 (K), J1.2 (Pin_2), J10.1 (Pin_1), J11.4 (Pin_4), J12.1 (Pin_1), J14.4 (Pin_4), J2.2 (Pin_2), J3.1 (Pin_1), J6.1 (Pin_1), J7.2 (Pin_2), R25.1, R4.1, R6.1, R9.1, U1.1 (IN)
- net GND: now also R2.2, A1.1 (GND), A1.7 (GND), A2.1 (GND), A2.7 (GND), A3.1 (GND), A3.7 (GND), A4.1 (GND), A4.7 (GND), C1.2, C10.2, C12.1, C14.2, C15.1, C2.2, C3.2, C4.2, C5.2, C6.2, C7.2, C8.2, D10.1 (K), J1.1 (Pin_1), J11.3 (Pin_3), J13.2 (Pin_2), J14.3 (Pin_3), J16.2 (Pin_2), J17.1 (Pin_1), J18.1 (Pin_1), J19.5, J23.1 (Pin_1), J24.1 (Pin_1), J25.1 (Pin_1), J26.1 (Pin_1), J4.2 (Pin_2), J5.2 (Pin_2), J8.1 (Pin_1), J8.3 (Pin_3), J8.5 (Pin_5), J8.7 (Pin_7), J9.2 (Pin_2), Q2.3 (S), Q3.3 (S), Q4.3 (S), R10.2, R11.1, R12.1, R19.2, R21.2, R24.2, R3.1, R5.2, R7.1, R8.2, U1.2 (GND), U3.15 (GND), U4.5 (GND); no longer R1.2
- net at Q1.1 (G): now also R2.1, J8.8 (Pin_8); no longer R1.1
- net at Q1.2 (D): now also D1.1 (K), D2.2 (A), J3.2 (Pin_2)
- new net: D3.1 (K), D4.2 (A), J6.2 (Pin_2), Q2.2 (D)
- new net: C6.1, J7.1 (Pin_1), J9.1 (Pin_1), R7.2
- new net: A3.12 (MS3), A3.13 (~{RESET}), A3.14 (~{SLEEP}), R15.1
- new net: C10.1, J14.1 (Pin_1), J16.1 (Pin_1), R12.2
- new net: R22.2, U5.1
- new net: R19.1, R22.1, U5.2 (-)
- new net: C15.2, R18.2, U5.3 (+)
- new net: A1.12 (MS3), A1.13 (~{RESET}), A1.14 (~{SLEEP}), R13.1
- new net: D5.1 (K), D6.2 (A), J10.2 (Pin_2), Q3.2 (D)
- new net: D10.2 (A), R25.2
- new net: D1.2 (A), R1.2
- new net: J8.2 (Pin_2), Q4.1 (G), R10.1
- new net: J8.4 (Pin_4), Q3.1 (G), R8.1
- new net: J8.6 (Pin_6), Q2.1 (G), R5.1
- new net: U2.10 (GND), U2.11 (GND)
- new net: R21.1, R23.1, U6.2 (-)
- new net: R23.2, U6.1
- new net: C13.1, U3.2 (VS+)
- new net: A1.3 (1B), J21.1 (Pin_1)
- new net: A1.4 (1A), J21.2 (Pin_2)
- new net: A1.5 (2A), J21.3 (Pin_3)
- new net: A1.6 (2B), J21.4 (Pin_4)
- new net: D7.2 (A), R9.2
- new net: D9.1 (K), R24.1
- new net: C7.1, J11.1 (Pin_1), J13.1 (Pin_1), R11.2
- new net: J25.2 (Pin_2), R17.1
- new net: C14.1, R17.2, R20.1
- new net: D5.2 (A), R6.2
- new net: A4.11 (MS2), J24.2 (Pin_2)
- new net: A4.10 (MS1), J24.3 (Pin_3)
- new net: A4.16 (DIR), J24.4 (Pin_4)
- new net: A4.15 (STEP), J24.5 (Pin_5)
- new net: A4.9 (~{ENABLE}), J24.6 (Pin_6)
- new net: C9.1, U3.1 (C1+)
- new net: J15.2 (Pin_2), U3.11 (T1IN)
- new net: J15.1 (Pin_1), U3.12 (R1OUT)
- new net: J19.3, U3.13 (R1IN)
- new net: J19.2, U3.14 (T1OUT)
- new net: C9.2, U3.3 (C1-)
- new net: C11.1, U3.4 (C2+)
- new net: C11.2, U3.5 (C2-)
- new net: C12.2, U3.6 (VS-)
- new net: A2.12 (MS3), A2.13 (~{RESET}), A2.14 (~{SLEEP}), R14.1
- new net: J20.1 (Pin_1), U4.4 (DI)
- new net: J20.2 (Pin_2), U4.3 (DE)
- new net: J20.3 (Pin_3), U4.2 (~{RE})
- new net: J20.4 (Pin_4), U4.1 (RO)
- new net: D3.2 (A), R4.2
- new net: J26.2 (Pin_2), R18.1
- new net: D7.1 (K), D8.2 (A), J12.2 (Pin_2), Q4.2 (D)
- new net: A4.12 (MS3), A4.13 (~{RESET}), A4.14 (~{SLEEP}), R16.1
- new net: A4.3 (1B), J28.1 (Pin_1)
- new net: A4.4 (1A), J28.2 (Pin_2)
- new net: A4.5 (2A), J28.3 (Pin_3)
- new net: A4.6 (2B), J28.4 (Pin_4)
- new net: A3.3 (1B), J27.1 (Pin_1)
- new net: A3.4 (1A), J27.2 (Pin_2)
- new net: A3.5 (2A), J27.3 (Pin_3)
- new net: A3.6 (2B), J27.4 (Pin_4)
- new net: C3.1, J2.1 (Pin_1), J4.1 (Pin_1), R3.2
- new net: A3.10 (MS1), J23.3 (Pin_3)
- new net: A3.11 (MS2), J23.2 (Pin_2)
- new net: A3.15 (STEP), J23.5 (Pin_5)
- new net: A3.16 (DIR), J23.4 (Pin_4)
- new net: A3.9 (~{ENABLE}), J23.6 (Pin_6)
- new net: A2.3 (1B), J22.1 (Pin_1)
- new net: A2.4 (1A), J22.2 (Pin_2)
- new net: A2.5 (2A), J22.3 (Pin_3)
- new net: A2.6 (2B), J22.4 (Pin_4)
- new net: R20.2, U6.3 (+)
- new net: A2.10 (MS1), J18.3 (Pin_3)
- new net: A2.11 (MS2), J18.2 (Pin_2)
- new net: A2.15 (STEP), J18.5 (Pin_5)
- new net: A2.16 (DIR), J18.4 (Pin_4)
- new net: A2.9 (~{ENABLE}), J18.6 (Pin_6)
- new net: A1.11 (MS2), J17.2 (Pin_2)
- new net: A1.10 (MS1), J17.3 (Pin_3)
- new net: A1.16 (DIR), J17.4 (Pin_4)
- new net: A1.15 (STEP), J17.5 (Pin_5)
- new net: A1.9 (~{ENABLE}), J17.6 (Pin_6)
- new net +24v: A1.8 (VMOT), A2.8 (VMOT), A3.8 (VMOT), A4.8 (VMOT)
- new net +5V: C13.2, C5.1, C8.1, D9.2 (A), J5.1 (Pin_1), U1.3 (OUT), U3.16 (VCC)
- new net +5v: A1.2 (VDD), A2.2 (VDD), A3.2 (VDD), A4.2 (VDD), R13.2, R14.2, R15.2, R16.2
Other:
- note added: "0-10V DC (J1 from CPU Unit PWM 10KHz)"
- note added: "0-10V PWM (J1 from CPU Unit)"
- note added: "4-20ma"
- note added: "Etage d'alimentation 24v - 5v"
- note added: "PT5402 (pressure sensor)"
- note added: "Pilotage EV 24V"
- note added: "Pilotage moteurs pas à pas"
- note added: "RS232"
- note added: "RS485"
- note added: "TN2115 (temperature sensor)"
- note added: "UART_RX"
- note added: "UART_TX"
- note added: "capa grd"
