File: PCB_Banc.kicad_pcb (KiCad board)
At the start: 2 copper layers, 216.5 x 144 mm, 73 parts, among them J1 Screw_Terminal_01x02, J10 Screw_Terminal_01x02, J11 Screw_Terminal_01x04, J12 Screw_Terminal_01x02, J13 Screw_Terminal_01x02, J14 Screw_Terminal_01x04, J15 Screw_Terminal_01x02, J16 Screw_Terminal_01x02, J17 Screw_Terminal_01x06, J18 Screw_Terminal_01x06, J2 Screw_Terminal_01x02, J20 Screw_Terminal_01x04, J21 Screw_Terminal_01x04, J22 Screw_Terminal_01x04, J23 Screw_Terminal_01x06, J24 Screw_Terminal_01x06, J25 Screw_Terminal_01x02, J26 Screw_Terminal_01x02, J27 Screw_Terminal_01x04, J28 Screw_Terminal_01x04, J3 Screw_Terminal_01x02, J4 Screw_Terminal_01x02, J5 Screw_Terminal_01x02, J6 Screw_Terminal_01x02, J7 Screw_Terminal_01x02, J8 Screw_Terminal_01x08, J9 Screw_Terminal_01x02, Q1 IRLZ44N, Q2 IRLZ44N, Q3 IRLZ44N, Q4 IRLZ44N, U1 L7805, U2 XTR111AxDGQ, U4 MAX1487E

Commit message: PCB valid prod
Parts:
- added C1: 0.33µF, Capacitor_THT:CP_Radial_D5.0mm_P2.50mm, F.Cu at (86.6, 56.6)
- added C10: 470n, Capacitor_SMD:C_0805_2012Metric_Pad1.18x1.45mm_HandSolder, F.Cu at (62.6, 115.3)
- added C11: 1µF, Capacitor_SMD:C_0805_2012Metric_Pad1.18x1.45mm_HandSolder, F.Cu at (84.5, 108.5)
- added C12: 1µF, Capacitor_SMD:C_0805_2012Metric_Pad1.18x1.45mm_HandSolder, F.Cu at (80.0, 108.5)
- added C13: 1µF, Capacitor_SMD:C_0805_2012Metric_Pad1.18x1.45mm_HandSolder, F.Cu at (93.0, 108.5)
- added C14: 2.2µF, Capacitor_SMD:C_0805_2012Metric_Pad1.18x1.45mm_HandSolder, F.Cu at (119.0, 100.9)
- added C15: 100nF, Capacitor_SMD:C_0805_2012Metric_Pad1.18x1.45mm_HandSolder, F.Cu at (103.6, 100.0)
- added C16: 470n, Capacitor_SMD:C_0805_2012Metric_Pad1.18x1.45mm_HandSolder, F.Cu at (62.3, 92.2)
- added C17: 470n, Capacitor_SMD:C_0805_2012Metric_Pad1.18x1.45mm_HandSolder, F.Cu at (61.9, 127.5)
- added C18: 470n, Capacitor_SMD:C_0805_2012Metric_Pad1.18x1.45mm_HandSolder, F.Cu at (62.8, 82.8)
- added C19: 470n, Capacitor_SMD:C_0805_2012Metric_Pad1.18x1.45mm_HandSolder, F.Cu at (62.8, 73.2)
- added C2: 470µ, Capacitor_THT:CP_Radial_D5.0mm_P2.50mm, F.Cu at (79.5, 56.1)
- added C20: 0.33µF, Capacitor_THT:CP_Radial_D5.0mm_P2.50mm, F.Cu at (114.8, 55.1)
- added C21: 0.1µ, Capacitor_SMD:C_0805_2012Metric_Pad1.18x1.45mm_HandSolder, F.Cu at (97.8, 61.6)
- added C3: 470n, Capacitor_SMD:C_0805_2012Metric_Pad1.18x1.45mm_HandSolder, F.Cu at (62.7, 64.3)
- added C4: 100n, Capacitor_SMD:C_0805_2012Metric_Pad1.18x1.45mm_HandSolder, F.Cu at (90.1, 65.7)
- added C5: 0.1µ, Capacitor_SMD:C_0805_2012Metric_Pad1.18x1.45mm_HandSolder, F.Cu at (118.6, 68.3)
- added C6: 470n, Capacitor_SMD:C_0805_2012Metric_Pad1.18x1.45mm_HandSolder, F.Cu at (62.7, 55.5)
- added C7: 470n, Capacitor_SMD:C_0805_2012Metric_Pad1.18x1.45mm_HandSolder, F.Cu at (62.2, 103.0)
- added C8: 1µF, Capacitor_SMD:C_0805_2012Metric_Pad1.18x1.45mm_HandSolder, F.Cu at (90.8, 122.7)
- added C9: 1µF, Capacitor_SMD:C_0805_2012Metric_Pad1.18x1.45mm_HandSolder, F.Cu at (88.8, 108.5)
- added D11: LED, LED_SMD:LED_0805_2012Metric_Pad1.15x1.40mm_HandSolder, F.Cu at (101.3, 61.5)
- added H1: MountingHole, MountingHole:MountingHole_3mm_Pad, F.Cu at (181.3, 71.2)
- added H2: MountingHole, MountingHole:MountingHole_3mm_Pad, F.Cu at (123.7, 84.5)
- added H3: MountingHole, MountingHole:MountingHole_3mm_Pad, F.Cu at (77.4, 65.2)
- added H4: MountingHole, MountingHole:MountingHole_3mm_Pad, F.Cu at (75.4, 125.2)
- added J19: Conn_01x01, Connector_PinSocket_2.54mm:PinSocket_1x01_P2.54mm_Vertical, F.Cu at (87.1, 94.2)
- added J29: Screw_Terminal_01x04, TerminalBlock_Phoenix:TerminalBlock_Phoenix_MPT-0,5-4-2.54_1x04_P2.54mm_Horizontal, F.Cu at (54.6, 88.5)
- added J30: Conn_01x04, Connector_PinSocket_2.54mm:PinSocket_1x04_P2.54mm_Vertical, F.Cu at (145.0, 105.0)
- added J31: Screw_Terminal_01x04, TerminalBlock_Phoenix:TerminalBlock_Phoenix_MPT-0,5-4-2.54_1x04_P2.54mm_Horizontal, F.Cu at (54.6, 124.7)
- added J32: Conn_01x01, Connector_PinSocket_2.54mm:PinSocket_1x01_P2.54mm_Vertical, F.Cu at (77.4, 78.4)
- added J33: Screw_Terminal_01x02, TerminalBlock_Phoenix:TerminalBlock_Phoenix_MPT-0,5-2-2.54_1x02_P2.54mm_Horizontal, F.Cu at (54.1, 73.3)
- added J35: Screw_Terminal_01x02, TerminalBlock_Phoenix:TerminalBlock_Phoenix_MPT-0,5-2-2.54_1x02_P2.54mm_Horizontal, F.Cu at (54.1, 66.3)
- added J37: ~, TerminalBlock_Phoenix:TerminalBlock_Phoenix_MPT-0,5-2-2.54_1x02_P2.54mm_Horizontal, F.Cu at (103.3, 54.1)
- added J39: Conn_01x02, Connector_PinSocket_2.54mm:PinSocket_1x02_P2.54mm_Vertical, F.Cu at (62.1, 61.0)
- added J40: Conn_01x02, Connector_PinSocket_2.54mm:PinSocket_1x02_P2.54mm_Vertical, F.Cu at (62.0, 52.3)
- added J41: Conn_01x02, Connector_PinSocket_2.54mm:PinSocket_1x02_P2.54mm_Vertical, F.Cu at (62.2, 79.5)
- added J42: Conn_01x02, Connector_PinSocket_2.54mm:PinSocket_1x02_P2.54mm_Vertical, F.Cu at (62.1, 69.9)
- added J43: Conn_01x02, Connector_PinSocket_2.54mm:PinSocket_1x02_P2.54mm_Vertical, F.Cu at (61.4, 112.2)
- added J44: Conn_01x02, Connector_PinSocket_2.54mm:PinSocket_1x02_P2.54mm_Vertical, F.Cu at (61.3, 88.8)
- added J45: Conn_01x03, Connector_PinSocket_2.54mm:PinSocket_1x03_P2.54mm_Vertical, F.Cu at (85.0, 133.3)
- added Q5: 2N3904, Package_TO_SOT_THT:TO-92_Inline, F.Cu at (91.6, 79.5)
- added Q6: 2N3904, Package_TO_SOT_THT:TO-92_Inline, F.Cu at (82.5, 80.0)
- added R26: 1K, Resistor_SMD:R_0805_2012Metric_Pad1.20x1.40mm_HandSolder, F.Cu at (62.3, 94.6)
- added R27: 1K, Resistor_SMD:R_0805_2012Metric_Pad1.20x1.40mm_HandSolder, F.Cu at (61.9, 130.0)
- added R28: 1k, Resistor_SMD:R_0805_2012Metric_Pad1.20x1.40mm_HandSolder, F.Cu at (62.8, 85.3)
- added R29: 1k, Resistor_SMD:R_0805_2012Metric_Pad1.20x1.40mm_HandSolder, F.Cu at (62.8, 76.2)
- added R30: 470, Resistor_SMD:R_0805_2012Metric_Pad1.20x1.40mm_HandSolder, F.Cu at (103.3, 61.5)
- added R31: 120, Resistor_SMD:R_0805_2012Metric_Pad1.20x1.40mm_HandSolder, F.Cu at (115.4, 121.0)
- added R32: 1k, Resistor_SMD:R_0805_2012Metric_Pad1.20x1.40mm_HandSolder, F.Cu at (110.9, 121.0)
- added R33: 1k, Resistor_SMD:R_0805_2012Metric_Pad1.20x1.40mm_HandSolder, F.Cu at (108.4, 124.0)
- added R34: 1K, Resistor_SMD:R_0805_2012Metric_Pad1.20x1.40mm_HandSolder, F.Cu at (62.2, 107.7)
- added R35: 1K, Resistor_SMD:R_0805_2012Metric_Pad1.20x1.40mm_HandSolder, F.Cu at (62.6, 119.8)
- added R36: 1K, Resistor_SMD:R_0805_2012Metric_Pad1.20x1.40mm_HandSolder, F.Cu at (62.3, 96.9)
- added R37: 1K, Resistor_SMD:R_0805_2012Metric_Pad1.20x1.40mm_HandSolder, F.Cu at (61.9, 132.3)
- added R38: 330, Resistor_SMD:R_0805_2012Metric_Pad1.20x1.40mm_HandSolder, F.Cu at (77.4, 82.5)
- added R39: 100, Resistor_SMD:R_0805_2012Metric_Pad1.20x1.40mm_HandSolder, F.Cu at (111.5, 76.4)
- added R40: 499, Resistor_SMD:R_0805_2012Metric_Pad1.20x1.40mm_HandSolder, F.Cu at (95.7, 83.5)
- added U3: MAX232, Package_SO:SOIC-16W_5.3x10.2mm_P1.27mm, F.Cu at (85.7, 114.8)
- added U5: LM358, Package_SO:SOIC-8-1EP_3.9x4.9mm_P1.27mm_EP2.29x3mm, F.Cu at (101.2, 108.1)
- added U6: LM358, Package_SO:SOIC-8-1EP_3.9x4.9mm_P1.27mm_EP2.29x3mm, F.Cu at (121.5, 112.8)
- added U7: LM7812_TO220, Package_TO_SOT_THT:TO-220-3_Vertical, F.Cu at (105.4, 70.4)
- D1, D10, D3, D5, D7, D9: footprint LED_SMD:LED_0201_0603Metric_Pad0.64x0.40mm_HandSolder -> LED_SMD:LED_0805_2012Metric_Pad1.15x1.40mm_HandSolder
- D2, D4, D6: footprint Diode_SMD:D_0805_2012Metric -> Diode_SMD:D_0805_2012Metric_Pad1.15x1.40mm_HandSolder
- J13, J16, J4: value Screw_Terminal_01x02 -> Conn_01x04; footprint TerminalBlock_Phoenix:TerminalBlock_Phoenix_MPT-0,5-2-2.54_1x02_P2.54mm_Horizontal -> Connector_PinSocket_2.54mm:PinSocket_1x04_P2.54mm_Vertical
- J15, J25, J26: value Screw_Terminal_01x02 -> Conn_01x02; footprint TerminalBlock_Phoenix:TerminalBlock_Phoenix_MPT-0,5-2-2.54_1x02_P2.54mm_Horizontal -> Connector_PinSocket_2.54mm:PinSocket_1x02_P2.54mm_Vertical
- J17, J18, J23, J24: value Screw_Terminal_01x06 -> Conn_01x02; footprint TerminalBlock_Phoenix:TerminalBlock_Phoenix_MPT-0,5-6-2.54_1x06_P2.54mm_Horizontal -> Connector_PinSocket_2.54mm:PinSocket_1x02_P2.54mm_Vertical
- J20: value Screw_Terminal_01x04 -> Conn_01x02; footprint TerminalBlock_Phoenix:TerminalBlock_Phoenix_MPT-0,5-4-2.54_1x04_P2.54mm_Horizontal -> Connector_PinSocket_2.54mm:PinSocket_1x02_P2.54mm_Vertical
- J21, J22, J27, J28: value Screw_Terminal_01x04 -> Conn_01x06; footprint TerminalBlock_Phoenix:TerminalBlock_Phoenix_MPT-0,5-4-2.54_1x04_P2.54mm_Horizontal -> Connector_PinSocket_2.54mm:PinSocket_1x06_P2.54mm_Vertical
- J5: value Screw_Terminal_01x02 -> Arduino pwr supply
- J8: value Screw_Terminal_01x08 -> Conn_01x04; footprint TerminalBlock_Phoenix:TerminalBlock_Phoenix_MPT-0,5-8-2.54_1x08_P2.54mm_Horizontal -> Connector_PinSocket_2.54mm:PinSocket_1x04_P2.54mm_Vertical
- J9: value Screw_Terminal_01x02 -> Conn_01x08; footprint TerminalBlock_Phoenix:TerminalBlock_Phoenix_MPT-0,5-2-2.54_1x02_P2.54mm_Horizontal -> Connector_PinSocket_2.54mm:PinSocket_1x08_P2.54mm_Vertical
- R10, R5, R6, R9: footprint Resistor_SMD:R_0805_2012Metric -> Resistor_SMD:R_0805_2012Metric_Pad1.20x1.40mm_HandSolder
- R11, R12, R13, R14, R15, R16, R17, R20, R21, R23: footprint Resistor_THT:R_Axial_DIN0411_L9.9mm_D3.6mm_P12.70mm_Horizontal -> Resistor_SMD:R_0805_2012Metric_Pad1.20x1.40mm_HandSolder
- R25: value 1k -> 2k
- R3, R7: value 247 -> 1k; footprint Resistor_THT:R_Axial_DIN0411_L9.9mm_D3.6mm_P12.70mm_Horizontal -> Resistor_SMD:R_0805_2012Metric_Pad1.20x1.40mm_HandSolder
- U2: value XTR111AxDGQ -> LM324; footprint Package_SO:MSOP-10-1EP_3x3mm_P0.5mm_EP2.2x3.1mm_Mask1.83x1.89mm_ThermalVias -> Package_SO:SOIC-14-16_3.9x9.9mm_P1.27mm
- moved J24 378.8 mm to (85.1, 122.3), turned to -90 degrees
- moved J18 373.4 mm to (61.7, 124.4), turned to 90 degrees
- moved J7 368.0 mm to (54.1, 52.3), turned to -90 degrees
- moved J17 362.9 mm to (61.2, 100.0), turned to 90 degrees
- moved J11 360.7 mm to (54.6, 100.5), turned to -90 degrees
- moved J14 360.7 mm to (54.6, 112.9), turned to -90 degrees
- moved J23 358.3 mm to (120.0, 94.9), turned to 90 degrees
- moved J2 344.7 mm to (54.1, 59.3), turned to -90 degrees
- moved J4 337.6 mm to (117.4, 133.3), turned to -90 degrees
- moved J13 332.1 mm to (145.9, 73.7), turned to -90 degrees
- moved R11 332.0 mm to (62.2, 105.5), turned to 180 degrees
- moved R7 331.7 mm to (62.7, 58.0), turned to 180 degrees
- moved R3 331.0 mm to (62.7, 66.8), turned to 180 degrees
- moved U2 326.7 mm to (86.6, 87.1), turned to -90 degrees
- moved J20 321.0 mm to (103.8, 95.0), turned to -90 degrees
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Connections:
- A1 pad 1: GND2 -> GND
- A1 pad 2: +5v -> +5V
- A1 pad 7: GND2 -> GND
- A1 pad 8: +24v -> +24V
- A2 pad 1: GND2 -> GND
- A2 pad 2: +5v -> +5V
- A2 pad 7: GND2 -> GND
- A2 pad 8: +24v -> +24V
- A3 pad 1: GND2 -> GND
- A3 pad 2: +5v -> +5V
- A3 pad 7: GND2 -> GND
- A3 pad 8: +24v -> +24V
- A4 pad 1: GND2 -> GND
- A4 pad 2: +5v -> +5V
- A4 pad 7: GND2 -> GND
- A4 pad 8: +24v -> +24V
- D9 pad 2: Net-(D9-A) -> +5V
- J1 pad 1: GND -> +24V
- J1 pad 2: +24V -> GND
- J11 pad 2: unconnected-(J11-Pin_2-Pad2) -> Net-(J11-Pin_2)
- J13 pad 1: Net-(J11-Pin_1) -> Net-(A3-1B)
- J13 pad 2: GND -> Net-(A3-1A)
- J14 pad 2: unconnected-(J14-Pin_2-Pad2) -> Net-(J14-Pin_2)
- J15 pad 2: Net-(J15-Pin_2) -> GND
- J16 pad 1: Net-(J14-Pin_1) -> Net-(A1-1B)
- J16 pad 2: GND -> Net-(A1-1A)
- J17 pad 1: GND2 -> Net-(J11-Pin_1)
- J17 pad 2: Net-(A1-MS2) -> GND
- J18 pad 1: GND2 -> Net-(J18-Pin_1)
- J18 pad 2: Net-(A2-MS2) -> GND
- J2 pad 2: +12V -> +24V
- J20 pad 1: Net-(J20-Pin_1) -> GND
- J21 pad 1: Net-(A1-1B) -> GND
- J21 pad 2: Net-(A1-1A) -> Net-(A2-MS2)
- J21 pad 3: Net-(A1-2A) -> Net-(A2-MS1)
- J21 pad 4: Net-(A1-2B) -> Net-(A2-DIR)
- J22 pad 1: Net-(A2-1B) -> GND
- J22 pad 2: Net-(A2-1A) -> Net-(A1-MS2)
- J22 pad 3: Net-(A2-2A) -> Net-(A1-MS1)
- J22 pad 4: Net-(A2-2B) -> Net-(A1-DIR)
- J23 pad 1: GND2 -> GND
- J23 pad 2: Net-(A3-MS2) -> Net-(J23-Pin_2)
- J24 pad 1: GND2 -> Net-(J24-Pin_1)
- J24 pad 2: Net-(A4-MS2) -> Net-(J24-Pin_2)
- J25 pad 1: GND -> Net-(J25-Pin_1)
- J25 pad 2: Net-(J25-Pin_2) -> GND
- J26 pad 1: GND -> Net-(J26-Pin_1)
- J26 pad 2: Net-(J26-Pin_2) -> GND
- J27 pad 1: Net-(A3-1B) -> GND
- J27 pad 2: Net-(A3-1A) -> Net-(A3-MS2)
- J27 pad 3: Net-(A3-2A) -> Net-(A3-MS1)
- J27 pad 4: Net-(A3-2B) -> Net-(A3-DIR)
- J28 pad 1: Net-(A4-1B) -> GND
- J28 pad 2: Net-(A4-1A) -> Net-(A4-MS2)
- J28 pad 3: Net-(A4-2A) -> Net-(A4-MS1)
- J28 pad 4: Net-(A4-2B) -> Net-(A4-DIR)
- J4 pad 1: Net-(J2-Pin_1) -> Net-(J4-Pin_1)
- J4 pad 2: GND -> Net-(J4-Pin_2)
- J5 pad 1: Net-(D9-A) -> +5V
- J7 pad 1: Net-(J7-Pin_1) -> Net-(J40-Pin_1)
- J7 pad 2: +12V -> +24V
- J8 pad 1: GND -> Net-(A2-1B)
- J8 pad 2: Net-(J8-Pin_2) -> Net-(A2-1A)
- J8 pad 3: GND -> Net-(A2-2A)
- J8 pad 4: Net-(J8-Pin_4) -> Net-(A2-2B)
- J9 pad 1: Net-(J7-Pin_1) -> GND
- J9 pad 2: GND -> Net-(J9-Pin_2)
- Q1 pad 1: Net-(J8-Pin_8) -> Net-(J9-Pin_8)
- Q1 pad 3: GND2 -> GND
- Q2 pad 1: Net-(J8-Pin_6) -> Net-(J9-Pin_6)
- Q2 pad 3: GND2 -> GND
- Q3 pad 1: Net-(J8-Pin_4) -> Net-(J9-Pin_4)
- Q3 pad 3: GND2 -> GND
- Q4 pad 1: Net-(J8-Pin_2) -> Net-(J9-Pin_2)
- Q4 pad 3: GND2 -> GND
- R10 pad 1: Net-(J8-Pin_2) -> Net-(J9-Pin_2)
- R10 pad 2: GND2 -> GND
- R13 pad 2: +5v -> +5V
- R14 pad 2: +5v -> +5V
- R15 pad 2: +5v -> +5V
- R16 pad 2: +5v -> +5V
- R17 pad 1: Net-(J25-Pin_2) -> Net-(J23-Pin_2)
- R18 pad 1: Net-(J26-Pin_2) -> Net-(J20-Pin_2)
- R2 pad 1: Net-(J8-Pin_8) -> Net-(J9-Pin_8)
- R2 pad 2: GND2 -> GND
- R22 pad 2: Net-(R22-Pad2) -> Net-(J25-Pin_1)
- R23 pad 2: Net-(R23-Pad2) -> Net-(J26-Pin_1)
- R5 pad 1: Net-(J8-Pin_6) -> Net-(J9-Pin_6)
- R5 pad 2: GND2 -> GND
- R7 pad 2: Net-(J7-Pin_1) -> Net-(J40-Pin_1)
- R8 pad 1: Net-(J8-Pin_4) -> Net-(J9-Pin_4)
- R8 pad 2: GND2 -> GND
- U1 pad 3: Net-(D9-A) -> +5V
- U2 pad 1: unconnected-(U2-VSP-Pad1) -> Net-(Q5-B)
- U2 pad 10: Net-(U2-GND-Pad10) -> (no net)
- U2 pad 11: Net-(U2-GND-Pad10) -> (no net)
- U2 pad 3: unconnected-(U2-VG-Pad3) -> Net-(J19-Pin_1)
- U2 pad 4: unconnected-(U2-REGS-Pad4) -> (no net)
- U2 pad 5: unconnected-(U2-REGF-Pad5) -> Net-(Q5-C)
- U2 pad 6: unconnected-(U2-VIN-Pad6) -> Net-(Q6-C)
- U2 pad 7: unconnected-(U2-SET-Pad7) -> Net-(Q6-B)
- U2 pad 8: unconnected-(U2-~{EF}-Pad8) -> (no net)
- U2 pad 9: unconnected-(U2-OD-Pad9) -> (no net)
- U4 pad 1: Net-(J20-Pin_4) -> Net-(J4-Pin_4)
- U4 pad 2: Net-(J20-Pin_3) -> Net-(J4-Pin_3)
- U4 pad 3: Net-(J20-Pin_2) -> Net-(J4-Pin_2)
- U4 pad 4: Net-(J20-Pin_1) -> Net-(J4-Pin_1)
- U4 pad 6: unconnected-(U4-A-Pad6) -> Net-(J15-Pin_1)
- U4 pad 7: unconnected-(U4-B-Pad7) -> Net-(U4-B)
- U4 pad 8: unconnected-(U4-VCC-Pad8) -> +5V
Routing:
- net +24V: track 0.00 -> 444.6 mm, vias 0 -> 5
- net +5V: track 0.00 -> 320.2 mm
- net Net-(Q6-C): track 0.00 -> 34.1 mm
- net Net-(A2-STEP): track 0.00 -> 28.1 mm
- net Net-(A1-STEP): track 0.00 -> 27.6 mm
- net Net-(A3-STEP): track 0.00 -> 27.4 mm
- net Net-(A4-STEP): track 0.00 -> 27.4 mm
- net GND: track 0.00 -> 27.4 mm, vias 0 -> 8
- net Net-(J9-Pin_2): track 0.00 -> 26.3 mm
- net Net-(U6A--): track 0.00 -> 21.6 mm
- net +12V: track 0.00 -> 21.4 mm
- net Net-(J9-Pin_8): track 0.00 -> 19.3 mm
- net Net-(J9-Pin_4): track 0.00 -> 18.0 mm
- net Net-(A2-DIR): track 0.00 -> 17.9 mm
- net Net-(A1-DIR): track 0.00 -> 17.4 mm
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- added copper zone on F.Cu, net +24V
- added copper zone on B.Cu, net GND
- added copper zone on F.Cu, net GND
Other:
- board size 216.5 x 144 mm -> 135.6 x 85.3 mm
